File: analog-photography/hardware/dispocam-hub/dispocam-hub.kicad_pcb (KiCad board)
At the start: 2 copper layers, 50.8 x 22.9 mm, 46 parts, among them J1 Conn_01x16, J2 Conn_01x12, M1 Motor_Servo_Pair, M2 Motor_Servo_Pair, M3 Motor_Servo_Pair, M4 Motor_Servo_Pair, SW1 Wind Limit, SW2 Wind Limit, SW3 Wind Limit, SW4 Wind Limit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

Commit message: finalize PCB design, export gerbers, clean up schematic
Other:
- rule pad_to_mask_clearance: 0.038 -> 0
Changed lines of the file:
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@@
       (dielectric_constraints no)
     )
-    (pad_to_mask_clearance 0.038)
+    (pad_to_mask_clearance 0)
+    (aux_axis_origin 119.38 91.44)
     (pcbplotparams
       (layerselection 0x00010fc_ffffffff)
@@
       (outputformat 1)
       (mirror false)
-      (drillshape 1)
+      (drillshape 0)
       (scaleselection 1)
-      (outputdirectory "")
+      (outputdirectory "gerbers/")
     )
   )
